File: arnogeddon_megalotone.kicad_pcb (KiCad board)
At the start: 2 copper layers, 59.7 x 38.1 mm, 28 parts, among them P1 IN L, P2 IN R, P3 OUT L, P4 OUT R, P5 9V Batt, SW1 mono, U1 TL072

Commit message: /**/
Parts:
- moved C8 23.3 mm to (193.0, 92.7)
- moved C10 16.3 mm to (203.2, 86.4), turned to 180 degrees
- moved RV2 15.5 mm to (177.8, 105.4)
- moved RV1 13.5 mm to (177.8, 102.9)
- moved C7 12.7 mm to (167.6, 92.7), turned to 180 degrees
- moved U1 6.48 mm to (177.8, 83.8)
- moved R3 2.84 mm to (151.1, 81.3), turned to 270 degrees
- moved R6 1.27 mm to (161.3, 74.9)
- turned R4 to 0 degrees
Other:
- net class Default: clearance 0.2 -> 0.254; trace_width 0.25 -> 0.381; via_dia 0.6 -> 0.762; via_drill 0.4 -> 0.508
- rule trace_clearance: 0.2 -> 0.254
Changed lines of the file:
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@@
     (links 44)
     (no_connects 44)
-    (area 146.05 68.58 207.01 107.95)
+    (area 146.05 67.31 207.01 110.49)
     (thickness 1.6)
     (drawings 4)
@@
   )
   (setup
-    (last_trace_width 0.25)
-    (trace_clearance 0.2)
+    (last_trace_width 0.381)
+    (trace_clearance 0.254)
     (zone_clearance 0.508)
     (zone_45_only no)
@@
     (segment_width 0.2)
     (edge_width 0.15)
-    (via_size 0.6)
-    (via_drill 0.4)
+    (via_size 0.762)
+    (via_drill 0.508)
     (via_min_size 0.4)
     (via_min_drill 0.3)
@@
   (net 19 "Net-(R8-Pad1)")
   (net_class Default "This is the default net class."
-    (clearance 0.2)
-    (trace_width 0.25)
-    (via_dia 0.6)
-    (via_drill 0.4)
+    (clearance 0.254)
+    (trace_width 0.381)
+    (via_dia 0.762)
+    (via_drill 0.508)
     (uvia_dia 0.3)
     (uvia_drill 0.1)
@@
   )
   (module Capacitors_Elko_ThroughHole:Elko_vert_DM6-3_RM2-5 placed (layer F.Cu)
-    (at 177.8 100.33)
+    (at 167.64 92.71 180)
     (descr "Electrolytic Capacitor, vertical, diameter 6,3mm, RM 2,5mm, radial,")
     (tags "Electrolytic Capacitor, vertical, diameter 6,3mm, RM 2,5mm, Elko, Electrolytkondensator, Kondensator gepolt, Durchmesser 6,3mm, radial,")
-    (fp_text reference C7 (at 0 -5.08) (layer F.SilkS)
-      (effects (font (thickness 0.3048)))
-    )
-    (fp_text value 47u (at 0 5.08) (layer F.SilkS) hide
+    (fp_text reference C7 (at 0 -5.08 180) (layer F.SilkS)
+      (effects (font (thickness 0.3048)))
+    )
+    (fp_text value 47u (at 0 5.08 180) (layer F.SilkS) hide
       (effects (font (thickness 0.3048)))
     )
@@
     (fp_line (start -1.00076 -1.30048) (end -1.00076 -1.19888) (layer F.Cu) (width 0.381))
     (fp_circle (center 0 0) (end 3.1496 0) (layer F.SilkS) (width 0.381))
-    (pad 2 thru_hole circle (at 1.27 0) (size 1.50114 1.50114) (drill 0.8001) (layers *.Cu *.Mask F.SilkS)
+    (pad 2 thru_hole circle (at 1.27 0 180) (size 1.50114 1.50114) (drill 0.8001) (layers *.Cu *.Mask F.SilkS)
       (net 9 "Net-(C7-Pad2)"))
-    (pad 1 thru_hole circle (at -1.27 0) (size 1.50114 1.50114) (drill 0.8001) (layers *.Cu *.Mask F.SilkS)
+    (pad 1 thru_hole circle (at -1.27 0 180) (size 1.50114 1.50114) (drill 0.8001) (layers *.Cu *.Mask F.SilkS)
       (net 10 "Net-(C7-Pad1)"))
   )
   (module Capacitors_Elko_ThroughHole:Elko_vert_DM6-3_RM2-5 placed (layer F.Cu)
-    (at 171.45 83.82)
+    (at 193.04 92.71)
     (descr "Electrolytic Capacitor, vertical, diameter 6,3mm, RM 2,5mm, radial,")
     (tags "Electrolytic Capacitor, vertical, diameter 6,3mm, RM 2,5mm, Elko, Electrolytkondensator, Kondensator gepolt, Durchmesser 6,3mm, radial,")
@@
   )
   (module Capacitors_Elko_ThroughHole:Elko_vert_DM7-5_RM2-5 placed (layer F.Cu)
-    (at 190.5 96.52)
+    (at 203.2 86.36 180)
     (descr "Electrolytic Capacitor, vertical, diameter 7,5mm, RM 2,5mm, radial,")
     (tags "Electrolytic Capacitor, vertical, diameter 7,5mm, RM 2,5mm, Elko, Electrolytkondensator, Kondensator gepolt, Durchmesser 7,5mm, radial,")
-    (fp_text reference C10 (at 0 -5.08) (layer F.SilkS)
-      (effects (font (thickness 0.3048)))
-    )
-    (fp_text value 100u (at 0 5.08) (layer F.SilkS) hide
+    (fp_text reference C10 (at 0 -5.08 180) (layer F.SilkS)
+      (effects (font (thickness 0.3048)))
+    )
+    (fp_text value 100u (at 0 5.08 180) (layer F.SilkS) hide
       (effects (font (thickness 0.3048)))
     )
@@
     (fp_line (start -2.413 -1.905) (end -1.27 -1.905) (layer F.Cu) (width 0.381))
     (fp_circle (center 0 0) (end 3.81 0) (layer F.SilkS) (width 0.381))
-    (pad 2 thru_hole circle (at 1.27 0) (size 1.50114 1.50114) (drill 0.8001) (layers *.Cu *.Mask F.SilkS)
-      (net 2 GND))
-    (pad 1 thru_hole circle (at -1.27 0) (size 1.50114 1.50114) (drill 0.8001) (layers *.Cu *.Mask F.SilkS)
+    (pad 2 thru_hole circle (at 1.27 0 180) (size 1.50114 1.50114) (drill 0.8001) (layers *.Cu *.Mask F.SilkS)
+      (net 2 GND))
+    (pad 1 thru_hole circle (at -1.27 0 180) (size 1.50114 1.50114) (drill 0.8001) (layers *.Cu *.Mask F.SilkS)
       (net 5 Vcc))
   )
@@
   )
   (module Custom:R3-LARGE_PADS placed (layer F.Cu)
-    (at 149.86 83.82 180)
-    (descr "Resitance 3 pas")
-    (tags R)
-    (autoplace_cost180 10)
-    (fp_text reference R3 (at 0 0 180) (layer F.SilkS)
-      (effects (font (size 1 1) (thickness 0.2032)))
-    )
-    (fp_text value 100K (at 0 0 180) (layer F.SilkS)
-      (effects (font (size 1 1) (thickness 0.2032)))
-    )
-    (fp_line (start -3.81 0) (end -3.302 0) (layer F.SilkS) (width 0.3048))
-    (fp_line (start 3.81 0) (end 3.302 0) (layer F.SilkS) (width 0.3048))
-    (fp_line (start 3.302 0) (end 3.302 -1.016) (layer F.SilkS) (width 0.3048))
-    (fp_line (start 3.302 -1.016) (end -3.302 -1.016) (layer F.SilkS) (width 0.3048))
-    (fp_line (start -3.302 -1.016) (end -3.302 1.016) (layer F.SilkS) (width 0.3048))
-    (fp_line (start -3.302 1.016) (end 3.302 1.016) (layer F.SilkS) (width 0.3048))
-    (fp_line (start 3.302 1.016) (end 3.302 0) (layer F.SilkS) (width 0.3048))
-    (fp_line (start -3.302 -0.508) (end -2.794 -1.016) (layer F.SilkS) (width 0.3048))
-    (pad 1 thru_hole circle (at -3.81 0 180) (size 1.778 1.778) (drill 0.8128) (layers *.Cu *.Mask F.SilkS)
+    (at 151.13 81.28 270)
+    (descr "Resitance 3 pas")
+    (tags R)
+    (autoplace_cost180 10)
+    (fp_text reference R3 (at 0 0 270) (layer F.SilkS)
+      (effects (font (size 1 1) (thickness 0.2032)))
+    )
+    (fp_text value 100K (at 0 0 270) (layer F.SilkS)
+      (effects (font (size 1 1) (thickness 0.2032)))
+    )
+    (fp_line (start -3.81 0) (end -3.302 0) (layer F.SilkS) (width 0.3048))
+    (fp_line (start 3.81 0) (end 3.302 0) (layer F.SilkS) (width 0.3048))
+    (fp_line (start 3.302 0) (end 3.302 -1.016) (layer F.SilkS) (width 0.3048))
+    (fp_line (start 3.302 -1.016) (end -3.302 -1.016) (layer F.SilkS) (width 0.3048))
+    (fp_line (start -3.302 -1.016) (end -3.302 1.016) (layer F.SilkS) (width 0.3048))
+    (fp_line (start -3.302 1.016) (end 3.302 1.016) (layer F.SilkS) (width 0.3048))
+    (fp_line (start 3.302 1.016) (end 3.302 0) (layer F.SilkS) (width 0.3048))
+    (fp_line (start -3.302 -0.508) (end -2.794 -1.016) (layer F.SilkS) (width 0.3048))
+    (pad 1 thru_hole circle (at -3.81 0 270) (size 1.778 1.778) (drill 0.8128) (layers *.Cu *.Mask F.SilkS)
       (net 10 "Net-(C7-Pad1)"))
-    (pad 2 thru_hole circle (at 3.81 0 180) (size 1.778 1.778) (drill 0.8128) (layers *.Cu *.Mask F.SilkS)
+    (pad 2 thru_hole circle (at 3.81 0 270) (size 1.778 1.778) (drill 0.8128) (layers *.Cu *.Mask F.SilkS)
       (net 16 "Net-(R1-Pad2)"))
     (model discret/resistor.wrl
@@
   )
   (module Custom:R3-LARGE_PADS placed (layer F.Cu)
-    (at 187.96 105.41 180)
-    (descr "Resitance 3 pas")
-    (tags R)
-    (autoplace_cost180 10)
-    (fp_text reference R4 (at 0 0 180) (layer F.SilkS)
-      (effects (font (size 1 1) (thickness 0.2032)))
-    )
-    (fp_text value 10K (at 0 0 180) (layer F.SilkS)
-      (effects (font (size 1 1) (thickness 0.2032)))
-    )
-    (fp_line (start -3.81 0) (end -3.302 0) (layer F.SilkS) (width 0.3048))
-    (fp_line (start 3.81 0) (end 3.302 0) (layer F.SilkS) (width 0.3048))
-    (fp_line (start 3.302 0) (end 3.302 -1.016) (layer F.SilkS) (width 0.3048))
-    (fp_line (start 3.302 -1.016) (end -3.302 -1.016) (layer F.SilkS) (width 0.3048))
-    (fp_line (start -3.302 -1.016) (end -3.302 1.016) (layer F.SilkS) (width 0.3048))
-    (fp_line (start -3.302 1.016) (end 3.302 1.016) (layer F.SilkS) (width 0.3048))
-    (fp_line (start 3.302 1.016) (end 3.302 0) (layer F.SilkS) (width 0.3048))
-    (fp_line (start -3.302 -0.508) (end -2.794 -1.016) (layer F.SilkS) (width 0.3048))
-    (pad 1 thru_hole circle (at -3.81 0 180) (size 1.778 1.778) (drill 0.8128) (layers *.Cu *.Mask F.SilkS)
+    (at 187.96 105.41)
+    (descr "Resitance 3 pas")
+    (tags R)
+    (autoplace_cost180 10)
+    (fp_text reference R4 (at 0 0) (layer F.SilkS)
+      (effects (font (size 1 1) (thickness 0.2032)))
+    )
+    (fp_text value 10K (at 0 0) (layer F.SilkS)
+      (effects (font (size 1 1) (thickness 0.2032)))
+    )
+    (fp_line (start -3.81 0) (end -3.302 0) (layer F.SilkS) (width 0.3048))
+    (fp_line (start 3.81 0) (end 3.302 0) (layer F.SilkS) (width 0.3048))
+    (fp_line (start 3.302 0) (end 3.302 -1.016) (layer F.SilkS) (width 0.3048))
+    (fp_line (start 3.302 -1.016) (end -3.302 -1.016) (layer F.SilkS) (width 0.3048))
+    (fp_line (start -3.302 -1.016) (end -3.302 1.016) (layer F.SilkS) (width 0.3048))
+    (fp_line (start -3.302 1.016) (end 3.302 1.016) (layer F.SilkS) (width 0.3048))
+    (fp_line (start 3.302 1.016) (end 3.302 0) (layer F.SilkS) (width 0.3048))
+    (fp_line (start -3.302 -0.508) (end -2.794 -1.016) (layer F.SilkS) (width 0.3048))
+    (pad 1 thru_hole circle (at -3.81 0) (size 1.778 1.778) (drill 0.8128) (layers *.Cu *.Mask F.SilkS)
       (net 17 "Net-(R4-Pad1)"))
-    (pad 2 thru_hole circle (at 3.81 0 180) (size 1.778 1.778) (drill 0.8128) (layers *.Cu *.Mask F.SilkS)
+    (pad 2 thru_hole circle (at 3.81 0) (size 1.778 1.778) (drill 0.8128) (layers *.Cu *.Mask F.SilkS)
       (net 14 "Net-(P3-Pad2)"))
     (model discret/resistor.wrl
@@
   )
   (module Custom:R3-LARGE_PADS placed (layer F.Cu)
-    (at 161.29 76.2)
+    (at 161.29 74.93)
     (descr "Resitance 3 pas")
     (tags R)
@@
   )
   (module Custom:SIL-3-LARGE_PADS placed (layer F.Cu)
-    (at 168.91 92.71)
+    (at 177.8 102.87)
     (descr "Connecteur 3 pins")
     (tags "CONN DEV")
@@
   )
   (module Custom:SIL-3-LARGE_PADS placed (layer F.Cu)
-    (at 180.34 90.17)
+    (at 177.8 105.41)
     (descr "Connecteur 3 pins")
     (tags "CONN DEV")
@@
   )
   (module Custom:DIP-8_LARGE_PADS placed (layer F.Cu)
-    (at 184.15 82.55)
+    (at 177.8 83.82)
     (descr "8 pins DIL package, elliptical pads")
     (tags DIL)
