File: arnogeddon_megalotone.sch (KiCad schematic (older format))
At the start: 28 parts, among them P1 IN L, P2 IN R, P3 OUT L, P4 OUT R, P5 9V Batt, SW1 mono, U1 TL072

Commit message: latest mods
Signed-off-by: Badscrew <badscrew@dolganoff.com>
Parts:
- added D1: LED, symbol LED
- added D2: D_Schottky, symbol D_Schottky
- added P6: IN B.Left, Pin_Headers:Pin_Header_Straight_1x02, symbol CONN_01X02
- added P7: IN B.Right, Pin_Headers:Pin_Header_Straight_1x02, symbol CONN_01X02
- added R12, R14: 1K, symbol R
- added R15: 10K, Custom:R3-LARGE_PADS, symbol R
- added SW2.1, SW2.2, SW2.3: boost, Custom:SIL-3-LARGE_PADS, symbol SWITCH_INV_SMALL
- added SW3.1, SW3.2: A / B, Custom:SIL-3-LARGE_PADS, symbol SWITCH_INV_SMALL
- P1: value IN L -> IN A.Left
- P2: value IN R -> IN A.Right
- R3, R7: value 100K -> 47K
- RV1, RV2: footprint Custom:SIL-3-LARGE_PADS -> (none)
Connections:
- net labels removed: vCC
- wire segments 65 -> 96
- no-connect marks 1 -> 2
Other:
- moved on the sheet: C10, C9, P1, P2, P3, P4, P5, R10, R4, R8, R9, SW1
